Commit message: [ver] Integrated gripper, octomap, camera on head

File: sawyer_moveit_config/srdf/sawyer.srdf.xacro (robot description, xacro)
@@ -5,4 +5,5 @@
   <xacro:arg name="electric_gripper" default="false"/>
   <xacro:arg name="controller_box" default="true"/>
+  <xacro:arg name="custom_gripper" default="false"/>
   <!--Base Sawyer Collisions-->
   <xacro:include filename="$(find sawyer_moveit_config)/srdf/sawyer_base.srdf.xacro" />
@@ -18,3 +19,8 @@
     <xacro:rethink_electric_gripper side="right"/>
   </xacro:if>
+  <disable_collisions link1="stp_021709TP00478_base" link2="gripper_tcp" reason="Never" />
+  <disable_collisions link1="stp_021709TP00478_base" link2="stp_021709TP00478_tip" reason="Never" />
+  <disable_collisions link1="right_hand" link2="stp_021709TP00478_base" reason="Never" />
+  <xacro:if value="$(arg custom_gripper)">
+  </xacro:if>
 </robot>

File: sawyer_moveit_config/srdf/sawyer_base.srdf.xacro (robot description, xacro)
@@ -35,8 +35,17 @@
         <joint name="right_j6" value="0" />
     </group_state>
+    <group_state name="pick_start" group="right_arm">
+        <joint name="right_j0" value="-1.9125" />
+        <joint name="right_j1" value="-0.4455" />
+        <joint name="right_j2" value="-1.36205" />
+        <joint name="right_j3" value="-2.1716" />
+        <joint name="right_j4" value="0.9732" />
+        <joint name="right_j5" value="1.6793" />
+        <joint name="right_j6" value="0.60250" />
+    </group_state>
     <!--VIRTUAL JOINT: Purpose: this element defines a virtual joint between a
     robot link and an external frame of reference (considered fixed with
     respect to the robot)-->
-    <virtual_joint name="world" type="fixed" parent_frame="world" child_link="base" />
+   <!--  <virtual_joint name="world" type="fixed" parent_frame="world" child_link="base" /> -->
     <!--DISABLE COLLISIONS: By default it is assumed that any link of the robot
     could potentially come into collision with any other link in the robot.
